Commit message: fix some bug

File: assets/urdf/piper_arm/piper_description.urdf (robot description, URDF)
Before this commit: robot piper, 11 links, 10 joints
Links:
- added link hithink_ee; visual sphere radius=0.01
Joints:
- added joint hithink_ee: type fixed, parent gripper_base, child hithink_ee, origin xyz=0 0 0.1 rpy=0 -1.5708 0
